Commit message: muchos cambios

File: src/myur3sim/myur3_description/urdf/myur3.urdf.xacro (robot description, xacro)
@@ -1,15 +1,22 @@
-<?xml version="1.0"?>
+<?xml version="1.0" ?>
 <robot xmlns:xacro="http://www.ros.org/wiki/xacro" name="robot">
-    <link name="world"/>
+    <link name="world" />
     <link name="pedestal">
         <inertial>
-            <origin xyz="0.0 0.0 0.5" rpy="0.0 0.0 0.0"/>
-            <mass value="20.0"/>
-            <inertia ixx="200.0" ixy="200.0" ixz="200.0" iyy="200.0" iyz="200.0" izz="200.0"/>
+            <origin xyz="0.0 0.0 0.5" rpy="0.0 0.0 0.0" />
+            <mass value="20.0" />
+            <inertia
+        ixx="200.0"
+        ixy="200.0"
+        ixz="200.0"
+        iyy="200.0"
+        iyz="200.0"
+        izz="200.0"
+      />
         </inertial>
         <visual>
-            <origin xyz="0.0 0.0 0.5" rpy="0.0 0.0 0.0"/>
+            <origin xyz="0.0 0.0 0.5" rpy="0.0 0.0 0.0" />
             <geometry>
-                <cylinder radius="0.1" length="1.0"/>
+                <cylinder radius="0.1" length="1.0" />
             </geometry>
             <material name="Gray">
@@ -18,7 +25,7 @@
         </visual>
         <collision>
-            <origin xyz="0.0 0.0 0.5" rpy="0.0 0.0 0.0"/>
+            <origin xyz="0.0 0.0 0.5" rpy="0.0 0.0 0.0" />
             <geometry>
-                <cylinder radius="0.1" length="1.0"/>
+                <cylinder radius="0.1" length="1.0" />
             </geometry>
         </collision>
@@ -30,19 +37,26 @@
     </gazebo>
     <joint name="world_joint" type="fixed">
-        <parent link="world"/>
-        <child link="pedestal"/>
-        <origin xyz="0 0 0" rpy="0 0 0"/>
+        <parent link="world" />
+        <child link="pedestal" />
+        <origin xyz="0 0 0" rpy="0 0 0" />
     </joint>
-    <xacro:arg name="transmission_hw_interface" default="hardware_interface/PositionJointInterface"/>
+    <xacro:arg
+    name="transmission_hw_interface"
+    default="hardware_interface/PositionJointInterface"
+  />
     <!-- common stuff -->
-    <xacro:include filename="$(find ur_description)/urdf/common.gazebo.xacro"/>
+    <xacro:include filename="$(find ur_description)/urdf/common.gazebo.xacro" />
     <!-- ur3 -->
-    <xacro:include filename="$(find ur_description)/urdf/ur3.urdf.xacro"/>
+    <xacro:include filename="$(find ur_description)/urdf/ur3.urdf.xacro" />
     <!-- arm -->
-    <xacro:ur3_robot prefix="" joint_limited="true" transmission_hw_interface="$(arg transmission_hw_interface)" />
+    <xacro:ur3_robot
+    prefix=""
+    joint_limited="true"
+    transmission_hw_interface="$(arg transmission_hw_interface)"
+  />
     <joint name="base_joint" type="fixed">
-        <parent link="pedestal"/>
-        <child link="base_link"/>
-        <origin xyz="0 0 1" rpy="0 0 0"/>
+        <parent link="pedestal" />
+        <child link="base_link" />
+        <origin xyz="0 0 1" rpy="0 0 0" />
     </joint>
 </robot>

File: src/universal_robot/ur_description/urdf/ur3_robot.urdf.xacro (robot description, xacro)
@@ -1,6 +1,8 @@
-<?xml version="1.0"?>
-<robot xmlns:xacro="http://wiki.ros.org/xacro"
-       name="ur3" >
-  <xacro:arg name="transmission_hw_interface" default="hardware_interface/PositionJointInterface"/>
+<?xml version="1.0" ?>
+<robot xmlns:xacro="http://wiki.ros.org/xacro" name="ur3">
+  <xacro:arg
+    name="transmission_hw_interface"
+    default="hardware_interface/PositionJointInterface"
+  />
   <!-- common stuff -->
   <xacro:include filename="$(find ur_description)/urdf/common.gazebo.xacro" />
@@ -8,5 +10,7 @@
   <xacro:include filename="$(find ur_description)/urdf/ur3.urdf.xacro" />
   <!-- arm -->
-  <xacro:ur3_robot prefix="" joint_limited="false"
+  <xacro:ur3_robot
+    prefix=""
+    joint_limited="false"
     transmission_hw_interface="$(arg transmission_hw_interface)"
   />
@@ -14,5 +18,5 @@
   <joint name="world_joint" type="fixed">
     <parent link="world" />
-    <child link = "base_link" />
+    <child link="base_link" />
     <origin xyz="0.0 0.0 0.0" rpy="0.0 0.0 0.0" />
   </joint>
